File: memory.sch (KiCad schematic (older format))
At the start: 9 parts, among them U5 IS42S16400J-xC

Commit message: updates
Changed lines of the file:
@@
 EESchema Schematic File Version 4
+LIBS:Raptor2000-cache
 EELAYER 29 0
 EELAYER END
 $Descr A4 11693 8268
 encoding utf-8
-Sheet 10 4
+Sheet 4 4
 Title ""
 Date ""
@@
 U 1 1 5CAC59FE
 P 4750 4050
-F 0 "R34" V 4554 4050 50  0000 C CNN
-F 1 "0" V 4645 4050 50  0000 C CNN
+F 0 "R34" V 4750 4050 50  0000 C CNN
+F 1 "0" V 4800 4150 50  0000 C CNN
 F 2 "Resistor_SMD:R_0603_1608Metric" H 4750 4050 50  0001 C CNN
 F 3 "~" H 4750 4050 50  0001 C CNN

Commit message: added nand flash, removed sd card. finished rtc circuit. added leds
Parts:
- added C14: 0.1, symbol Device:C
- added R4: 10k, symbol Device:R_Small
- added U3: TC58CVG2S0HRAIG, symbol Exodus_Peripherals:TC58CVG2S0HRAIG
Connections:
- net labels added: EPIOS[0..31], FLASH_DAT0, FLASH_DAT1, FLASH_DAT2, FLASH_DAT3, FLASH_SCLK, ~FLASH_CS
- wire segments 104 -> 119
Other:
- moved on the sheet: R34

Commit message: added component values for RAM decoupling caps
Parts:
- C33, C34, C35, C36, C37, C38, C39: value C_Small -> 0.1u
Changed lines of the file:
@@
 P 7800 1500
 F 0 "C34" H 7892 1546 50  0000 L CNN
-F 1 "C_Small" H 7892 1455 50  0000 L CNN
+F 1 "0.1u" H 7892 1455 50  0000 L CNN
 F 2 "Capacitor_SMD:C_0603_1608Metric" H 7800 1500 50  0001 C CNN
 F 3 "~" H 7800 1500 50  0001 C CNN
@@
 P 8250 1500
 F 0 "C35" H 8342 1546 50  0000 L CNN
-F 1 "C_Small" H 8342 1455 50  0000 L CNN
+F 1 "0.1u" H 8342 1455 50  0000 L CNN
 F 2 "Capacitor_SMD:C_0603_1608Metric" H 8250 1500 50  0001 C CNN
 F 3 "~" H 8250 1500 50  0001 C CNN
@@
 P 8650 1500
 F 0 "C36" H 8742 1546 50  0000 L CNN
-F 1 "C_Small" H 8742 1455 50  0000 L CNN
+F 1 "0.1u" H 8742 1455 50  0000 L CNN
 F 2 "Capacitor_SMD:C_0603_1608Metric" H 8650 1500 50  0001 C CNN
 F 3 "~" H 8650 1500 50  0001 C CNN
@@
 P 9100 1500
 F 0 "C37" H 9192 1546 50  0000 L CNN
-F 1 "C_Small" H 9192 1455 50  0000 L CNN
+F 1 "0.1u" H 9192 1455 50  0000 L CNN
 F 2 "Capacitor_SMD:C_0603_1608Metric" H 9100 1500 50  0001 C CNN
 F 3 "~" H 9100 1500 50  0001 C CNN
@@
 P 9550 1500
 F 0 "C38" H 9642 1546 50  0000 L CNN
-F 1 "C_Small" H 9642 1455 50  0000 L CNN
+F 1 "0.1u" H 9642 1455 50  0000 L CNN
 F 2 "Capacitor_SMD:C_0603_1608Metric" H 9550 1500 50  0001 C CNN
 F 3 "~" H 9550 1500 50  0001 C CNN
@@
 P 9950 1500
 F 0 "C39" H 10042 1546 50  0000 L CNN
-F 1 "C_Small" H 10042 1455 50  0000 L CNN
+F 1 "0.1u" H 10042 1455 50  0000 L CNN
 F 2 "Capacitor_SMD:C_0603_1608Metric" H 9950 1500 50  0001 C CNN
 F 3 "~" H 9950 1500 50  0001 C CNN
@@
 P 7350 1500
 F 0 "C33" H 7442 1546 50  0000 L CNN
-F 1 "C_Small" H 7442 1455 50  0000 L CNN
+F 1 "0.1u" H 7442 1455 50  0000 L CNN
 F 2 "Capacitor_SMD:C_0603_1608Metric" H 7350 1500 50  0001 C CNN
 F 3 "~" H 7350 1500 50  0001 C CNN

Commit message: fixed misnamed EPI nets.
Connections:
- net labels added: EPI0S0, EPI0S1, EPI0S10, EPI0S11, EPI0S12, EPI0S13, EPI0S14, EPI0S15, EPI0S16, EPI0S17, EPI0S18, EPI0S19, EPI0S2, EPI0S28, EPI0S29, EPI0S3, EPI0S30, EPI0S31, EPI0S4, EPI0S5, EPI0S6, EPI0S7, EPI0S8, EPI0S9, EPI0S[0..31]
- net labels removed: EPIOS0, EPIOS1, EPIOS10, EPIOS11, EPIOS12, EPIOS13, EPIOS14, EPIOS15, EPIOS16, EPIOS17, EPIOS18, EPIOS19, EPIOS2, EPIOS28, EPIOS29, EPIOS3, EPIOS30, EPIOS31, EPIOS4, EPIOS5, EPIOS6, EPIOS7, EPIOS8, EPIOS9, EPIOS[0..31]
Changed lines of the file:
@@
 	3850 2200 3750 2200
 Text Label 3950 2350 0    50   ~ 0
-EPIOS13
+EPI0S13
 Text Label 3950 2450 0    50   ~ 0
-EPIOS14
+EPI0S14
 Text Label 3950 2550 0    50   ~ 0
-EPIOS0
+EPI0S0
 Text Label 3950 2650 0    50   ~ 0
-EPIOS1
+EPI0S1
 Text Label 3950 2750 0    50   ~ 0
-EPIOS2
+EPI0S2
 Text Label 3950 2850 0    50   ~ 0
-EPIOS3
+EPI0S3
 Text Label 3950 2950 0    50   ~ 0
-EPIOS4
+EPI0S4
 Text Label 3950 3050 0    50   ~ 0
-EPIOS5
+EPI0S5
 Text Label 3950 3150 0    50   ~ 0
-EPIOS6
+EPI0S6
 Text Label 3950 3250 0    50   ~ 0
-EPIOS7
+EPI0S7
 Text Label 3950 3350 0    50   ~ 0
-EPIOS8
+EPI0S8
 Text Label 3950 3450 0    50   ~ 0
-EPIOS9
+EPI0S9
 Text Label 3950 3550 0    50   ~ 0
-EPIOS10
+EPI0S10
 Text Label 3950 3650 0    50   ~ 0
-EPIOS11
+EPI0S11
 Text Label 3950 3750 0    50   ~ 0
-EPIOS12
+EPI0S12
 Text Label 3950 3850 0    50   ~ 0
-EPIOS29
+EPI0S29
 Text Label 3950 3950 0    50   ~ 0
-EPIOS30
+EPI0S30
 Text Label 3950 4050 0    50   ~ 0
-EPIOS31
+EPI0S31
 Text Label 3950 4150 0    50   ~ 0
-EPIOS16
+EPI0S16
 Text Label 3950 4250 0    50   ~ 0
-EPIOS17
+EPI0S17
 Text Label 3950 4350 0    50   ~ 0
-EPIOS28
+EPI0S28
 Text Label 3950 4450 0    50   ~ 0
-EPIOS18
+EPI0S18
 Text Label 3950 4550 0    50   ~ 0
-EPIOS19
+EPI0S19
 Wire Wire Line
 	6600 2350 7350 2350
@@
 	7350 3850 7450 3950
 Text Label 7050 2350 0    50   ~ 0
-EPIOS0
+EPI0S0
 Text Label 7050 2450 0    50   ~ 0
-EPIOS1
+EPI0S1
 Text Label 7050 2550 0    50   ~ 0
-EPIOS2
+EPI0S2
 Text Label 7050 2650 0    50   ~ 0
-EPIOS3
+EPI0S3
 Text Label 7050 2750 0    50   ~ 0
-EPIOS4
+EPI0S4
 Text Label 7050 2850 0    50   ~ 0
-EPIOS5
+EPI0S5
 Text Label 7050 2950 0    50   ~ 0
-EPIOS6
+EPI0S6
 Text Label 7050 3050 0    50   ~ 0
-EPIOS7
+EPI0S7
 Text Label 7050 3150 0    50   ~ 0
-EPIOS8
+EPI0S8
 Text Label 7050 3250 0    50   ~ 0
-EPIOS9
+EPI0S9
 Text Label 7000 3350 0    50   ~ 0
-EPIOS10
+EPI0S10
 Text Label 7000 3450 0    50   ~ 0
-EPIOS11
+EPI0S11
 Text Label 7000 3550 0    50   ~ 0
-EPIOS12
+EPI0S12
 Text Label 7000 3650 0    50   ~ 0
-EPIOS13
+EPI0S13
 Text Label 7000 3750 0    50   ~ 0
-EPIOS14
+EPI0S14
 Text Label 7000 3850 0    50   ~ 0
-EPIOS15
+EPI0S15
 Text HLabel 3750 2200 0    50   Input ~ 0
-EPIOS[0..31]
+EPI0S[0..31]
 Wire Wire Line
 	9300 2650 9300 2800

Commit message: fixed component value for decoupling cap on nand flash.
Parts:
- C14: value 0.1 -> 0.1u
Changed lines of the file:
@@
 P 10500 3050
 F 0 "C14" H 10615 3096 50  0000 L CNN
-F 1 "0.1" H 10615 3005 50  0000 L CNN
+F 1 "0.1u" H 10615 3005 50  0000 L CNN
 F 2 "" H 10538 2900 50  0001 C CNN
 F 3 "~" H 10500 3050 50  0001 C CNN

Commit message: Fixed some componenet values. Added some layout notes. added decoupling cap to usb-to-uart circuit.
Parts:
- added R22, R24: DNP, symbol Device:R_Small
- added R23: 1M, symbol Device:R_Small
Connections:
- wire segments 119 -> 131
Other:
- note added: "EPI Traces must have a capacitance of < 35pF"
Changed lines of the file:
@@
 	1    0    0    -1
 $EndComp
-Wire Wire Line
-	9200 2800 9300 2800
-Wire Wire Line
-	9300 2450 9300 2350
 $Comp
 L power:+3.3V #PWR0120
 U 1 1 5D35E492
-P 9300 2350
-F 0 "#PWR0120" H 9300 2200 50  0001 C CNN
-F 1 "+3.3V" H 9315 2523 50  0000 C CNN
-F 2 "" H 9300 2350 50  0001 C CNN
-F 3 "" H 9300 2350 50  0001 C CNN
-	1    9300 2350
-	1    0    0    -1
-$EndComp
-Wire Wire Line
-	9400 3100 9200 3100
-Wire Wire Line
-	9400 2900 9200 2900
-Wire Wire Line
-	9400 3000 9200 3000
-Wire Wire Line
-	9400 3300 9200 3300
-Wire Wire Line
-	9400 3200 9200 3200
-Text HLabel 9200 3100 0    50   Input ~ 0
+P 9050 2250
+F 0 "#PWR0120" H 9050 2100 50  0001 C CNN
+F 1 "+3.3V" H 9065 2423 50  0000 C CNN
+F 2 "" H 9050 2250 50  0001 C CNN
+F 3 "" H 9050 2250 50  0001 C CNN
+	1    9050 2250
+	1    0    0    -1
+$EndComp
+Text HLabel 8750 3100 0    50   Input ~ 0
 FLASH_DAT0
-Text HLabel 9200 2900 0    50   Input ~ 0
+Text HLabel 8750 2900 0    50   Input ~ 0
 FLASH_DAT1
-Text HLabel 9200 3000 0    50   Input ~ 0
+Text HLabel 8750 3000 0    50   Input ~ 0
 FLASH_DAT2
-Text HLabel 9200 3200 0    50   Input ~ 0
+Text HLabel 8750 3200 0    50   Input ~ 0
 FLASH_SCLK
-Text HLabel 9200 3300 0    50   Input ~ 0
+Text HLabel 8750 3300 0    50   Input ~ 0
 FLASH_DAT3
-Text HLabel 9200 2800 0    50   Input ~ 0
+Text HLabel 8750 2800 0    50   Input ~ 0
 ~FLASH_CS
-Connection ~ 9300 2800
 Wire Wire Line
 	9300 2800 9400 2800
@@
 Wire Wire Line
 	9300 2650 9300 2800
+Wire Wire Line
+	8750 3300 8800 3300
+Wire Wire Line
+	8750 3200 9000 3200
+Wire Wire Line
+	8750 3100 9400 3100
+Wire Wire Line
+	8750 3000 9050 3000
+Wire Wire Line
+	8750 2900 9400 2900
+Wire Wire Line
+	8750 2800 9300 2800
+Connection ~ 9300 2800
+$Comp
+L Device:R_Small R22
+U 1 1 5D15943F
+P 8800 2550
+F 0 "R22" H 8859 2596 50  0000 L CNN
+F 1 "DNP" H 8859 2505 50  0000 L CNN
+F 2 "" H 8800 2550 50  0001 C CNN
+F 3 "~" H 8800 2550 50  0001 C CNN
+	1    8800 2550
+	1    0    0    -1
+$EndComp
+$Comp
+L Device:R_Small R23
+U 1 1 5D15A674
+P 9000 3500
+F 0 "R23" H 9059 3546 50  0000 L CNN
+F 1 "1M" H 9059 3455 50  0000 L CNN
+F 2 "" H 9000 3500 50  0001 C CNN
+F 3 "~" H 9000 3500 50  0001 C CNN
+	1    9000 3500
+	1    0    0    -1
+$EndComp
+Wire Wire Line
+	9050 2650 9050 3000
+Connection ~ 9050 3000
+Wire Wire Line
+	9050 3000 9400 3000
+Wire Wire Line
+	8800 2650 8800 3300
+Connection ~ 8800 3300
+Wire Wire Line
+	8800 3300 9400 3300
+Wire Wire Line
+	9000 3400 9000 3200
+Connection ~ 9000 3200
+Wire Wire Line
+	9000 3200 9400 3200
+Wire Wire Line
+	9050 2450 9050 2300
+Wire Wire Line
+	9050 2300 9300 2300
+Wire Wire Line
+	9300 2300 9300 2450
+Connection ~ 9050 2300
+Wire Wire Line
+	9050 2300 8800 2300
+Wire Wire Line
+	8800 2300 8800 2450
+Wire Wire Line
+	9050 2250 9050 2300
+Wire Wire Line
+	9000 3600 9000 3700
 Wire Bus Line
 	7450 2300 7450 5350
 Wire Bus Line
 	3850 2200 3850 5350
+$Comp
+L power:GND #PWR0144
+U 1 1 5D17FF4A
+P 9000 3700
+F 0 "#PWR0144" H 9000 3450 50  0001 C CNN
+F 1 "GND" H 9005 3527 50  0000 C CNN
+F 2 "" H 9000 3700 50  0001 C CNN
+F 3 "" H 9000 3700 50  0001 C CNN
+	1    9000 3700
+	1    0    0    -1
+$EndComp
+$Comp
+L Device:R_Small R24
+U 1 1 5D158F93
+P 9050 2550
+F 0 "R24" H 9109 2596 50  0000 L CNN
+F 1 "DNP" H 9109 2505 50  0000 L CNN
+F 2 "" H 9050 2550 50  0001 C CNN
+F 3 "~" H 9050 2550 50  0001 C CNN
+	1    9050 2550
+	1    0    0    -1
+$EndComp
+Text Notes 3200 2100 0    50   ~ 0
+EPI Traces must have a capacitance of < 35pF
 $EndSCHEMATC

Commit message: added part footprints. added usb-uart leds.
Parts:
- C14: footprint (none) -> Capacitor_SMD:C_0603_1608Metric
- R22, R23, R24, R4: footprint (none) -> Resistor_SMD:R_0603_1608Metric
- U3: footprint (none) -> Exodus_Packages:WSON-8-1EP_3.4x4.3mm_P1.27mm
Changed lines of the file:
@@
 F 0 "U3" H 9900 3565 50  0000 C CNN
 F 1 "TC58CVG2S0HRAIG" H 9900 3474 50  0000 C CNN
-F 2 "" H 9900 3000 50  0001 C CNN
+F 2 "Exodus_Packages:WSON-8-1EP_3.4x4.3mm_P1.27mm" H 9900 3000 50  0001 C CNN
 F 3 "" H 9900 3000 50  0001 C CNN
 	1    9900 3050
@@
 F 0 "C14" H 10615 3096 50  0000 L CNN
 F 1 "0.1u" H 10615 3005 50  0000 L CNN
-F 2 "" H 10538 2900 50  0001 C CNN
+F 2 "Capacitor_SMD:C_0603_1608Metric" H 10538 2900 50  0001 C CNN
 F 3 "~" H 10500 3050 50  0001 C CNN
 	1    10500 3050
@@
 F 0 "R4" H 9359 2596 50  0000 L CNN
 F 1 "10k" H 9359 2505 50  0000 L CNN
-F 2 "" H 9300 2550 50  0001 C CNN
+F 2 "Resistor_SMD:R_0603_1608Metric" H 9300 2550 50  0001 C CNN
 F 3 "~" H 9300 2550 50  0001 C CNN
 	1    9300 2550
@@
 F 0 "R22" H 8859 2596 50  0000 L CNN
 F 1 "DNP" H 8859 2505 50  0000 L CNN
-F 2 "" H 8800 2550 50  0001 C CNN
+F 2 "Resistor_SMD:R_0603_1608Metric" H 8800 2550 50  0001 C CNN
 F 3 "~" H 8800 2550 50  0001 C CNN
 	1    8800 2550
@@
 F 0 "R23" H 9059 3546 50  0000 L CNN
 F 1 "1M" H 9059 3455 50  0000 L CNN
-F 2 "" H 9000 3500 50  0001 C CNN
+F 2 "Resistor_SMD:R_0603_1608Metric" H 9000 3500 50  0001 C CNN
 F 3 "~" H 9000 3500 50  0001 C CNN
 	1    9000 3500
@@
 Wire Wire Line
 	9000 3600 9000 3700
-Wire Bus Line
-	7450 2300 7450 5350
-Wire Bus Line
-	3850 2200 3850 5350
 $Comp
 L power:GND #PWR0144
@@
 F 0 "R24" H 9109 2596 50  0000 L CNN
 F 1 "DNP" H 9109 2505 50  0000 L CNN
-F 2 "" H 9050 2550 50  0001 C CNN
+F 2 "Resistor_SMD:R_0603_1608Metric" H 9050 2550 50  0001 C CNN
 F 3 "~" H 9050 2550 50  0001 C CNN
 	1    9050 2550
@@
 Text Notes 3200 2100 0    50   ~ 0
 EPI Traces must have a capacitance of < 35pF
+Wire Bus Line
+	7450 2300 7450 5350
+Wire Bus Line
+	3850 2200 3850 5350
 $EndSCHEMATC
