File: memory.sch (KiCad schematic (older format))
At the start: 15 parts, among them U3 TC58CVG2S0HRAIG, U5 IS42S16400J-xC

Commit message: regenerated netlist/annotations and refdeses. using new connector symbol.
Parts:
- renumbered C33 to C201, C34 to C202, C35 to C203, C36 to C204, C37 to C205, C38 to C206, C39 to C207, C14 to C208, R34 to R201, R22 to R202, R23 to R203, R24 to R204, R4 to R205, U5 to U201, U3 to U202
Changed lines of the file:
@@
 	6000 4900 6000 5000
 $Comp
-L Device:R_Small R34
+L Device:R_Small R201
 U 1 1 5CAC59FE
 P 4500 4050
-F 0 "R34" V 4500 4050 50  0000 C CNN
+F 0 "R201" V 4500 4050 50  0000 C CNN
 F 1 "0" V 4550 4150 50  0000 C CNN
 F 2 "Resistor_SMD:R_0603_1608Metric" H 4500 4050 50  0001 C CNN
@@
 $EndComp
 $Comp
-L Exodus_Memory_RAM:IS42S16400J-xC U5
+L Exodus_Memory_RAM:IS42S16400J-xC U201
 U 1 1 5CAC8069
 P 5800 3450
-F 0 "U5" H 5800 5028 50  0000 C CNN
+F 0 "U201" H 5800 5028 50  0000 C CNN
 F 1 "IS42S16400J-xC" H 5800 4937 50  0000 C CNN
 F 2 "Package_SO:TSOP-II-54_22.2x10.16mm_P0.8mm" H 5800 3450 50  0001 C CNN
@@
 	5850 5000 6000 5000
 $Comp
-L power:GND #PWR0188
+L power:GND #PWR0202
 U 1 1 5CB12768
 P 5850 5100
-F 0 "#PWR0188" H 5850 4850 50  0001 C CNN
+F 0 "#PWR0202" H 5850 4850 50  0001 C CNN
 F 1 "GND" H 5855 4927 50  0000 C CNN
 F 2 "" H 5850 5100 50  0001 C CNN
@@
 $EndComp
 $Comp
-L power:+3.3V #PWR0189
+L power:+3.3V #PWR0201
 U 1 1 5CB1282D
 P 5850 1650
-F 0 "#PWR0189" H 5850 1500 50  0001 C CNN
+F 0 "#PWR0201" H 5850 1500 50  0001 C CNN
 F 1 "+3.3V" H 5865 1823 50  0000 C CNN
 F 2 "" H 5850 1650 50  0001 C CNN
@@
 	5850 1750 6000 1750
 $Comp
-L Device:C_Small C34
+L Device:C_Small C202
 U 1 1 5CB18DA3
 P 7800 1500
-F 0 "C34" H 7892 1546 50  0000 L CNN
+F 0 "C202" H 7892 1546 50  0000 L CNN
 F 1 "0.1u" H 7892 1455 50  0000 L CNN
 F 2 "Capacitor_SMD:C_0603_1608Metric" H 7800 1500 50  0001 C CNN
@@
 $EndComp
 $Comp
-L Device:C_Small C35
+L Device:C_Small C203
 U 1 1 5CB18E2B
 P 8250 1500
-F 0 "C35" H 8342 1546 50  0000 L CNN
+F 0 "C203" H 8342 1546 50  0000 L CNN
 F 1 "0.1u" H 8342 1455 50  0000 L CNN
 F 2 "Capacitor_SMD:C_0603_1608Metric" H 8250 1500 50  0001 C CNN
@@
 $EndComp
 $Comp
-L Device:C_Small C36
+L Device:C_Small C204
 U 1 1 5CB18E5B
 P 8650 1500
-F 0 "C36" H 8742 1546 50  0000 L CNN
+F 0 "C204" H 8742 1546 50  0000 L CNN
 F 1 "0.1u" H 8742 1455 50  0000 L CNN
 F 2 "Capacitor_SMD:C_0603_1608Metric" H 8650 1500 50  0001 C CNN
@@
 $EndComp
 $Comp
-L Device:C_Small C37
+L Device:C_Small C205
 U 1 1 5CB18F6F
 P 9100 1500
-F 0 "C37" H 9192 1546 50  0000 L CNN
+F 0 "C205" H 9192 1546 50  0000 L CNN
 F 1 "0.1u" H 9192 1455 50  0000 L CNN
 F 2 "Capacitor_SMD:C_0603_1608Metric" H 9100 1500 50  0001 C CNN
@@
 $EndComp
 $Comp
-L Device:C_Small C38
+L Device:C_Small C206
 U 1 1 5CB18F76
 P 9550 1500
-F 0 "C38" H 9642 1546 50  0000 L CNN
+F 0 "C206" H 9642 1546 50  0000 L CNN
 F 1 "0.1u" H 9642 1455 50  0000 L CNN
 F 2 "Capacitor_SMD:C_0603_1608Metric" H 9550 1500 50  0001 C CNN
@@
 $EndComp
 $Comp
-L Device:C_Small C39
+L Device:C_Small C207
 U 1 1 5CB18F7D
 P 9950 1500
-F 0 "C39" H 10042 1546 50  0000 L CNN
+F 0 "C207" H 10042 1546 50  0000 L CNN
 F 1 "0.1u" H 10042 1455 50  0000 L CNN
 F 2 "Capacitor_SMD:C_0603_1608Metric" H 9950 1500 50  0001 C CNN
@@
 $EndComp
 $Comp
-L Device:C_Small C33
+L Device:C_Small C201
 U 1 1 5CB1AA5F
 P 7350 1500
-F 0 "C33" H 7442 1546 50  0000 L CNN
+F 0 "C201" H 7442 1546 50  0000 L CNN
 F 1 "0.1u" H 7442 1455 50  0000 L CNN
 F 2 "Capacitor_SMD:C_0603_1608Metric" H 7350 1500 50  0001 C CNN
@@
 	7800 1300 8250 1300
 $Comp
-L power:+3.3V #PWR0190
+L power:+3.3V #PWR0203
 U 1 1 5CB33C9E
 P 8650 1150
-F 0 "#PWR0190" H 8650 1000 50  0001 C CNN
+F 0 "#PWR0203" H 8650 1000 50  0001 C CNN
 F 1 "+3.3V" H 8665 1323 50  0000 C CNN
 F 2 "" H 8650 1150 50  0001 C CNN
@@
 	8650 1150 8650 1300
 $Comp
-L power:GND #PWR0191
+L power:GND #PWR0204
 U 1 1 5CB365F7
 P 8650 1850
-F 0 "#PWR0191" H 8650 1600 50  0001 C CNN
+F 0 "#PWR0204" H 8650 1600 50  0001 C CNN
 F 1 "GND" H 8655 1677 50  0000 C CNN
 F 2 "" H 8650 1850 50  0001 C CNN
@@
 CLK
 $Comp
-L Exodus_Peripherals:TC58CVG2S0HRAIG U3
+L Exodus_Peripherals:TC58CVG2S0HRAIG U202
 U 1 1 5D346BB9
 P 9900 3050
-F 0 "U3" H 9900 3565 50  0000 C CNN
+F 0 "U202" H 9900 3565 50  0000 C CNN
 F 1 "TC58CVG2S0HRAIG" H 9900 3474 50  0000 C CNN
 F 2 "Exodus_Packages:WSON-8-1EP_3.4x4.3mm_P1.27mm" H 9900 3000 50  0001 C CNN
@@
 	10500 3300 10500 3450
 $Comp
-L power:GND #PWR0118
+L power:GND #PWR0208
 U 1 1 5D34E798
 P 10500 3450
-F 0 "#PWR0118" H 10500 3200 50  0001 C CNN
+F 0 "#PWR0208" H 10500 3200 50  0001 C CNN
 F 1 "GND" H 10505 3277 50  0000 C CNN
 F 2 "" H 10500 3450 50  0001 C CNN
@@
 $EndComp
 $Comp
-L power:+3.3V #PWR0119
+L power:+3.3V #PWR0207
 U 1 1 5D34EBD4
 P 10500 2650
-F 0 "#PWR0119" H 10500 2500 50  0001 C CNN
+F 0 "#PWR0207" H 10500 2500 50  0001 C CNN
 F 1 "+3.3V" H 10515 2823 50  0000 C CNN
 F 2 "" H 10500 2650 50  0001 C CNN
@@
 $EndComp
 $Comp
-L Device:C C14
+L Device:C C208
 U 1 1 5D351BF7
 P 10500 3050
-F 0 "C14" H 10615 3096 50  0000 L CNN
+F 0 "C208" H 10615 3096 50  0000 L CNN
 F 1 "0.1u" H 10615 3005 50  0000 L CNN
 F 2 "Capacitor_SMD:C_0603_1608Metric" H 10538 2900 50  0001 C CNN
@@
 Connection ~ 10500 3300
 $Comp
-L Device:R_Small R4
+L Device:R_Small R205
 U 1 1 5D357E46
 P 9300 2550
-F 0 "R4" H 9359 2596 50  0000 L CNN
+F 0 "R205" H 9359 2596 50  0000 L CNN
 F 1 "10k" H 9359 2505 50  0000 L CNN
 F 2 "Resistor_SMD:R_0603_1608Metric" H 9300 2550 50  0001 C CNN
@@
 $EndComp
 $Comp
-L power:+3.3V #PWR0120
+L power:+3.3V #PWR0206
 U 1 1 5D35E492
 P 9050 2250
-F 0 "#PWR0120" H 9050 2100 50  0001 C CNN
+F 0 "#PWR0206" H 9050 2100 50  0001 C CNN
 F 1 "+3.3V" H 9065 2423 50  0000 C CNN
 F 2 "" H 9050 2250 50  0001 C CNN
@@
 Connection ~ 9300 2800
 $Comp
-L Device:R_Small R22
+L Device:R_Small R202
 U 1 1 5D15943F
 P 8800 2550
-F 0 "R22" H 8859 2596 50  0000 L CNN
+F 0 "R202" H 8859 2596 50  0000 L CNN
 F 1 "DNP" H 8859 2505 50  0000 L CNN
 F 2 "Resistor_SMD:R_0603_1608Metric" H 8800 2550 50  0001 C CNN
@@
 $EndComp
 $Comp
-L Device:R_Small R23
+L Device:R_Small R203
 U 1 1 5D15A674
 P 9000 3500
-F 0 "R23" H 9059 3546 50  0000 L CNN
+F 0 "R203" H 9059 3546 50  0000 L CNN
 F 1 "1M" H 9059 3455 50  0000 L CNN
 F 2 "Resistor_SMD:R_0603_1608Metric" H 9000 3500 50  0001 C CNN
@@
 	9000 3600 9000 3700
 $Comp
-L power:GND #PWR0144
+L power:GND #PWR0205
 U 1 1 5D17FF4A
 P 9000 3700
-F 0 "#PWR0144" H 9000 3450 50  0001 C CNN
+F 0 "#PWR0205" H 9000 3450 50  0001 C CNN
 F 1 "GND" H 9005 3527 50  0000 C CNN
 F 2 "" H 9000 3700 50  0001 C CNN
@@
 $EndComp
 $Comp
-L Device:R_Small R24
+L Device:R_Small R204
 U 1 1 5D158F93
 P 9050 2550
-F 0 "R24" H 9109 2596 50  0000 L CNN
+F 0 "R204" H 9109 2596 50  0000 L CNN
 F 1 "DNP" H 9109 2505 50  0000 L CNN
 F 2 "Resistor_SMD:R_0603_1608Metric" H 9050 2550 50  0001 C CNN
