File: tm4c129.sch (KiCad schematic (older format))
At the start: 41 parts, among them U1 TM4C1294NCPDTGOOD, Y1 Crystal_GND24, Y2 Crystal

Commit message: updated come component values.
Parts:
- C10, C13, C15, C16: value 0.1 -> 0.1u
Changed lines of the file:
@@
 P 1950 1900
 F 0 "C10" H 2042 1946 50  0000 L CNN
-F 1 "0.1" H 2042 1855 50  0000 L CNN
+F 1 "0.1u" H 2042 1855 50  0000 L CNN
 F 2 "Capacitor_SMD:C_0603_1608Metric" H 1950 1900 50  0001 C CNN
 F 3 "~" H 1950 1900 50  0001 C CNN
@@
 P 2150 1250
 F 0 "C13" H 2242 1296 50  0000 L CNN
-F 1 "0.1" H 2242 1205 50  0000 L CNN
+F 1 "0.1u" H 2242 1205 50  0000 L CNN
 F 2 "Capacitor_SMD:C_0603_1608Metric" H 2150 1250 50  0001 C CNN
 F 3 "~" H 2150 1250 50  0001 C CNN
@@
 P 8050 3000
 F 0 "C15" V 8279 3000 50  0000 C CNN
-F 1 "0.1" V 8188 3000 50  0000 C CNN
+F 1 "0.1u" V 8188 3000 50  0000 C CNN
 F 2 "" H 8050 3000 50  0001 C CNN
 F 3 "~" H 8050 3000 50  0001 C CNN
@@
 P 8050 3350
 F 0 "C16" V 8279 3350 50  0000 C CNN
-F 1 "0.1" V 8188 3350 50  0000 C CNN
+F 1 "0.1u" V 8188 3350 50  0000 C CNN
 F 2 "" H 8050 3350 50  0001 C CNN
 F 3 "~" H 8050 3350 50  0001 C CNN
@@
 Wire Wire Line
 	5150 3650 5900 3650
-Wire Wire Line
-	5150 1350 5400 1350
-Text HLabel 5400 1350 2    50   Input ~ 0
+Text HLabel 5450 1350 2    50   Input ~ 0
 ~SYSRESET
 Wire Wire Line
@@
 Text Label 5450 2350 0    50   ~ 0
 EPI029
+Text Notes 6050 5050 0    50   ~ 0
+EPI0S31 should be configured for 12mA drive. \nThe rest of the EPI signals can be 8mA drive.
+Wire Wire Line
+	5150 1350 5450 1350
 Wire Bus Line
 	1700 4850 1700 7600
 Wire Bus Line
 	6000 2200 6000 7600
-Text Notes 6050 5050 0    50   ~ 0
-EPI0S31 should be configured for 12mA drive. \nThe rest of the EPI signals can be 8mA drive.
 $EndSCHEMATC

Commit message: added reset button and pullup. Moved sysreset to a gpio pin.
Connections:
- wire segments 222 -> 226
Other:
- note added: "Bulk Cap should total 2.2uF to 22uF"
- note added: "Ethernet Pull-up Resistors"
- note added: "Ethernet and User-Defined LEDs"
- note added: "Place Decoupling caps \nclose to power pairs"
- note added: "RC time circuit to meet ontime requirements"
- note added: "VDDC Decoupling cap should \ntotal 3.3uF to 3.4uF"
- moved on the sheet: C1, C10, C11, C12, C15, C16, C2, C3, C4, C5, C6, C7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

Commit message: added a debug microusb port.
Parts:
- added C?: 0.1u, symbol Device:C_Small
- added R?: 100, symbol Device:R_Small
- added R?: 10k, symbol Device:R_Small
- added SW?: RST_SW, symbol Switch:SW_Push
Connections:
- net labels added: UART_DEBUG_RXD, UART_DEBUG_TXD, ~RST
- wire segments 226 -> 246
Changed lines of the file:
@@
 $Descr A4 11693 8268
 encoding utf-8
-Sheet 4 4
+Sheet 4 5
 Title "TM4C129"
 Date "2019-06-22"
@@
 P 1550 4250
 F 0 "Y1" V 1504 4491 50  0000 L CNN
-F 1 "Crystal_GND24" V 1950 4250 50  0000 L CNN
+F 1 "Crystal_GND24" V 1400 4250 50  0000 L CNN
 F 2 "Crystal:Crystal_SMD_3225-4Pin_3.2x2.5mm" H 1550 4250 50  0001 C CNN
 F 3 "~" H 1550 4250 50  0001 C CNN
@@
 Wire Wire Line
 	5150 3650 5900 3650
-Text HLabel 5450 1350 2    50   Input ~ 0
-~SYSRESET
 Wire Wire Line
 	5150 5950 5400 5950
@@
 Wire Wire Line
 	1600 2350 1700 2350
+Text Label 5450 1350 2    50   ~ 0
+~RST
+$Comp
+L Switch:SW_Push SW?
+U 1 1 5D500B16
+P 7950 3050
+F 0 "SW?" V 7996 3198 50  0000 L CNN
+F 1 "RST_SW" V 7905 3198 50  0000 L CNN
+F 2 "" H 7950 3250 50  0001 C CNN
+F 3 "~" H 7950 3250 50  0001 C CNN
+	1    7950 3050
+	0    1    -1   0
+$EndComp
+$Comp
+L Device:R_Small R?
+U 1 1 5D5021C3
+P 7750 2750
+F 0 "R?" V 7554 2750 50  0000 C CNN
+F 1 "100" V 7645 2750 50  0000 C CNN
+F 2 "" H 7750 2750 50  0001 C CNN
+F 3 "~" H 7750 2750 50  0001 C CNN
+	1    7750 2750
+	0    -1   1    0
+$EndComp
+$Comp
+L Device:C_Small C?
+U 1 1 5D50D384
+P 7450 2950
+F 0 "C?" H 7358 2996 50  0000 R CNN
+F 1 "0.1u" H 7358 2905 50  0000 R CNN
+F 2 "" H 7450 2950 50  0001 C CNN
+F 3 "~" H 7450 2950 50  0001 C CNN
+	1    7450 2950
+	-1   0    0    -1
+$EndComp
+Wire Wire Line
+	7950 2850 7950 2750
+Wire Wire Line
+	7950 2750 7850 2750
+Wire Wire Line
+	7650 2750 7500 2750
+Wire Wire Line
+	7450 2750 7450 2850
+Wire Wire Line
+	7450 3050 7450 3350
+Wire Wire Line
+	7450 3350 7700 3350
+Wire Wire Line
+	7950 3350 7950 3250
+Wire Wire Line
+	7500 2750 7500 2650
+Connection ~ 7500 2750
+Wire Wire Line
+	7500 2750 7450 2750
+$Comp
+L Device:R_Small R?
+U 1 1 5D54D687
+P 7500 2550
+F 0 "R?" H 7441 2504 50  0000 R CNN
+F 1 "10k" H 7441 2595 50  0000 R CNN
+F 2 "" H 7500 2550 50  0001 C CNN
+F 3 "~" H 7500 2550 50  0001 C CNN
+	1    7500 2550
+	1    0    0    1
+$EndComp
+Wire Wire Line
+	7500 2450 7500 2400
+$Comp
+L power:+3.3V #PWR?
+U 1 1 5D55E558
+P 7500 2400
+F 0 "#PWR?" H 7500 2250 50  0001 C CNN
+F 1 "+3.3V" H 7515 2573 50  0000 C CNN
+F 2 "" H 7500 2400 50  0001 C CNN
+F 3 "" H 7500 2400 50  0001 C CNN
+	1    7500 2400
+	-1   0    0    -1
+$EndComp
+Wire Wire Line
+	7450 2750 7100 2750
+Connection ~ 7450 2750
+Wire Wire Line
+	7700 3350 7700 3400
+Connection ~ 7700 3350
+Wire Wire Line
+	7700 3350 7950 3350
+$Comp
+L power:GND #PWR?
+U 1 1 5D57F82F
+P 7700 3400
+F 0 "#PWR?" H 7700 3150 50  0001 C CNN
+F 1 "GND" H 7705 3227 50  0000 C CNN
+F 2 "" H 7700 3400 50  0001 C CNN
+F 3 "" H 7700 3400 50  0001 C CNN
+	1    7700 3400
+	-1   0    0    -1
+$EndComp
+Text Label 7100 2750 0    50   ~ 0
+~RST
+Wire Wire Line
+	5150 6050 5400 6050
+Text HLabel 5400 6050 2    50   Input ~ 0
+~SYSRESET
+Text HLabel 2450 4600 0    50   Input ~ 0
+UART_DEBUG_RXD
+Text HLabel 2450 4700 0    50   Input ~ 0
+UART_DEBUG_TXD
+Wire Wire Line
+	2550 4350 2550 4600
+Wire Wire Line
+	2550 4600 2450 4600
+Wire Wire Line
+	2550 4350 2750 4350
+Wire Wire Line
+	2600 4450 2600 4700
+Wire Wire Line
+	2600 4700 2450 4700
+Wire Wire Line
+	2600 4450 2750 4450
 Wire Bus Line
 	1700 4850 1700 7600

Commit message: Fixed some componenet values. Added some layout notes. added decoupling cap to usb-to-uart circuit.
Parts:
- R14: value 49.4 -> 49.9
- gave numbers to parts that had none: 4
Connections:
- wire segments 246 -> 248
Changed lines of the file:
@@
 P 8800 1300
 F 0 "R14" V 8996 1300 50  0000 C CNN
-F 1 "49.4" V 8905 1300 50  0000 C CNN
+F 1 "49.9" V 8905 1300 50  0000 C CNN
 F 2 "" H 8800 1300 50  0001 C CNN
 F 3 "~" H 8800 1300 50  0001 C CNN
@@
 ~RST
 $Comp
-L Switch:SW_Push SW?
+L Switch:SW_Push SW1
 U 1 1 5D500B16
 P 7950 3050
-F 0 "SW?" V 7996 3198 50  0000 L CNN
+F 0 "SW1" V 7996 3198 50  0000 L CNN
 F 1 "RST_SW" V 7905 3198 50  0000 L CNN
 F 2 "" H 7950 3250 50  0001 C CNN
@@
 $EndComp
 $Comp
-L Device:R_Small R?
+L Device:R_Small R18
 U 1 1 5D5021C3
 P 7750 2750
-F 0 "R?" V 7554 2750 50  0000 C CNN
+F 0 "R18" V 7554 2750 50  0000 C CNN
 F 1 "100" V 7645 2750 50  0000 C CNN
 F 2 "" H 7750 2750 50  0001 C CNN
@@
 $EndComp
 $Comp
-L Device:C_Small C?
+L Device:C_Small C17
 U 1 1 5D50D384
 P 7450 2950
-F 0 "C?" H 7358 2996 50  0000 R CNN
+F 0 "C17" H 7358 2996 50  0000 R CNN
 F 1 "0.1u" H 7358 2905 50  0000 R CNN
 F 2 "" H 7450 2950 50  0001 C CNN
@@
 	7500 2750 7450 2750
 $Comp
-L Device:R_Small R?
+L Device:R_Small R17
 U 1 1 5D54D687
 P 7500 2550
-F 0 "R?" H 7441 2504 50  0000 R CNN
+F 0 "R17" H 7441 2504 50  0000 R CNN
 F 1 "10k" H 7441 2595 50  0000 R CNN
 F 2 "" H 7500 2550 50  0001 C CNN
@@
 	7500 2450 7500 2400
 $Comp
-L power:+3.3V #PWR?
+L power:+3.3V #PWR0133
 U 1 1 5D55E558
 P 7500 2400
-F 0 "#PWR?" H 7500 2250 50  0001 C CNN
+F 0 "#PWR0133" H 7500 2250 50  0001 C CNN
 F 1 "+3.3V" H 7515 2573 50  0000 C CNN
 F 2 "" H 7500 2400 50  0001 C CNN
@@
 	7700 3350 7950 3350
 $Comp
-L power:GND #PWR?
+L power:GND #PWR0134
 U 1 1 5D57F82F
 P 7700 3400
-F 0 "#PWR?" H 7700 3150 50  0001 C CNN
+F 0 "#PWR0134" H 7700 3150 50  0001 C CNN
 F 1 "GND" H 7705 3227 50  0000 C CNN
 F 2 "" H 7700 3400 50  0001 C CNN
@@
 Wire Wire Line
 	2600 4450 2750 4450
+Wire Wire Line
+	5150 1250 5600 1250
+Wire Wire Line
+	5600 1250 5600 1300
 Wire Bus Line
 	1700 4850 1700 7600
 Wire Bus Line
 	6000 2200 6000 7600
+$Comp
+L power:GND #PWR0145
+U 1 1 5D1349D0
+P 5600 1300
+F 0 "#PWR0145" H 5600 1050 50  0001 C CNN
+F 1 "GND" H 5605 1127 50  0000 C CNN
+F 2 "" H 5600 1300 50  0001 C CNN
+F 3 "" H 5600 1300 50  0001 C CNN
+	1    5600 1300
+	1    0    0    -1
+$EndComp
 $EndSCHEMATC

Commit message: added part footprints. added usb-uart leds.
Parts:
- C15, C16, C17: footprint (none) -> Capacitor_SMD:C_0603_1608Metric
- D1, D2, D3, D4, D6, D7: footprint (none) -> LED_SMD:LED_0805_2012Metric
- D5: footprint LED_SMD:LED_0603_1608Metric -> LED_SMD:LED_0805_2012Metric
- R11, R12, R13, R14, R15, R16, R17, R18, R5, R7, R8, R9: footprint (none) -> Resistor_SMD:R_0603_1608Metric
- SW1: footprint (none) -> Button_Switch_SMD:SW_SPST_B3S-1000
- Y2: footprint (none) -> Crystal:Crystal_SMD_MicroCrystal_CC7V-T1A-2Pin_3.2x1.5mm
Changed lines of the file:
@@
 F 0 "Y2" V 6054 1231 50  0000 L CNN
 F 1 "Crystal" V 6145 1231 50  0000 L CNN
-F 2 "" H 6100 1100 50  0001 C CNN
+F 2 "Crystal:Crystal_SMD_MicroCrystal_CC7V-T1A-2Pin_3.2x1.5mm" H 6100 1100 50  0001 C CNN
 F 3 "~" H 6100 1100 50  0001 C CNN
 	1    6100 1100
@@
 F 0 "R5" V 8300 4600 50  0000 C CNN
 F 1 "330" V 8200 4600 50  0000 C CNN
-F 2 "" H 8100 4600 50  0001 C CNN
+F 2 "Resistor_SMD:R_0603_1608Metric" H 8100 4600 50  0001 C CNN
 F 3 "~" H 8100 4600 50  0001 C CNN
 	1    8100 4600
@@
 F 0 "D1" V 8139 4083 50  0000 R CNN
 F 1 "LED" V 8048 4083 50  0000 R CNN
-F 2 "" H 8100 4200 50  0001 C CNN
+F 2 "LED_SMD:LED_0805_2012Metric" H 8100 4200 50  0001 C CNN
 F 3 "~" H 8100 4200 50  0001 C CNN
 	1    8100 4200
@@
 F 0 "R7" V 8300 5900 50  0000 C CNN
 F 1 "330" V 8200 5900 50  0000 C CNN
-F 2 "" H 8100 5900 50  0001 C CNN
+F 2 "Resistor_SMD:R_0603_1608Metric" H 8100 5900 50  0001 C CNN
 F 3 "~" H 8100 5900 50  0001 C CNN
 	1    8100 5900
@@
 F 0 "D2" V 8139 5383 50  0000 R CNN
 F 1 "LED" V 8048 5383 50  0000 R CNN
-F 2 "" H 8100 5500 50  0001 C CNN
+F 2 "LED_SMD:LED_0805_2012Metric" H 8100 5500 50  0001 C CNN
 F 3 "~" H 8100 5500 50  0001 C CNN
 	1    8100 5500
@@
 F 0 "D3" V 9089 4083 50  0000 R CNN
 F 1 "LED" V 8998 4083 50  0000 R CNN
-F 2 "" H 9050 4200 50  0001 C CNN
+F 2 "LED_SMD:LED_0805_2012Metric" H 9050 4200 50  0001 C CNN
 F 3 "~" H 9050 4200 50  0001 C CNN
 	1    9050 4200
@@
 F 0 "R9" V 9250 5900 50  0000 C CNN
 F 1 "330" V 9150 5900 50  0000 C CNN
-F 2 "" H 9050 5900 50  0001 C CNN
+F 2 "Resistor_SMD:R_0603_1608Metric" H 9050 5900 50  0001 C CNN
 F 3 "~" H 9050 5900 50  0001 C CNN
 	1    9050 5900
@@
 F 0 "D4" V 9089 5383 50  0000 R CNN
 F 1 "LED" V 8998 5383 50  0000 R CNN
-F 2 "" H 9050 5500 50  0001 C CNN
+F 2 "LED_SMD:LED_0805_2012Metric" H 9050 5500 50  0001 C CNN
 F 3 "~" H 9050 5500 50  0001 C CNN
 	1    9050 5500
@@
 F 0 "D5" H 10142 2595 50  0000 C CNN
 F 1 "LED" H 10142 2686 50  0000 C CNN
-F 2 "LED_SMD:LED_0603_1608Metric" H 10150 2850 50  0001 C CNN
+F 2 "LED_SMD:LED_0805_2012Metric" H 10150 2850 50  0001 C CNN
 F 3 "~" H 10150 2850 50  0001 C CNN
 	1    10150 2850
@@
 F 0 "R8" V 9250 4600 50  0000 C CNN
 F 1 "330" V 9150 4600 50  0000 C CNN
-F 2 "" H 9050 4600 50  0001 C CNN
+F 2 "Resistor_SMD:R_0603_1608Metric" H 9050 4600 50  0001 C CNN
 F 3 "~" H 9050 4600 50  0001 C CNN
 	1    9050 4600
@@
 F 0 "D6" V 10189 4083 50  0000 R CNN
 F 1 "LED" V 10098 4083 50  0000 R CNN
-F 2 "" H 10150 4200 50  0001 C CNN
+F 2 "LED_SMD:LED_0805_2012Metric" H 10150 4200 50  0001 C CNN
 F 3 "~" H 10150 4200 50  0001 C CNN
 	1    10150 4200
@@
 F 0 "R12" V 10350 5900 50  0000 C CNN
 F 1 "330" V 10250 5900 50  0000 C CNN
-F 2 "" H 10150 5900 50  0001 C CNN
+F 2 "Resistor_SMD:R_0603_1608Metric" H 10150 5900 50  0001 C CNN
 F 3 "~" H 10150 5900 50  0001 C CNN
 	1    10150 5900
@@
 F 0 "D7" V 10189 5383 50  0000 R CNN
 F 1 "LED" V 10098 5383 50  0000 R CNN
-F 2 "" H 10150 5500 50  0001 C CNN
+F 2 "LED_SMD:LED_0805_2012Metric" H 10150 5500 50  0001 C CNN
 F 3 "~" H 10150 5500 50  0001 C CNN
 	1    10150 5500
@@
 F 0 "R11" V 10350 4600 50  0000 C CNN
 F 1 "330" V 10250 4600 50  0000 C CNN
-F 2 "" H 10150 4600 50  0001 C CNN
+F 2 "Resistor_SMD:R_0603_1608Metric" H 10150 4600 50  0001 C CNN
 F 3 "~" H 10150 4600 50  0001 C CNN
 	1    10150 4600
@@
 F 0 "R16" V 8996 1900 50  0000 C CNN
 F 1 "49.9" V 8905 1900 50  0000 C CNN
-F 2 "" H 8800 1900 50  0001 C CNN
+F 2 "Resistor_SMD:R_0603_1608Metric" H 8800 1900 50  0001 C CNN
 F 3 "~" H 8800 1900 50  0001 C CNN
 	1    8800 1900
@@
 F 0 "R15" V 8996 1600 50  0000 C CNN
 F 1 "49.9" V 8905 1600 50  0000 C CNN
-F 2 "" H 8800 1600 50  0001 C CNN
+F 2 "Resistor_SMD:R_0603_1608Metric" H 8800 1600 50  0001 C CNN
 F 3 "~" H 8800 1600 50  0001 C CNN
 	1    8800 1600
@@
 F 0 "R14" V 8996 1300 50  0000 C CNN
 F 1 "49.9" V 8905 1300 50  0000 C CNN
-F 2 "" H 8800 1300 50  0001 C CNN
+F 2 "Resistor_SMD:R_0603_1608Metric" H 8800 1300 50  0001 C CNN
 F 3 "~" H 8800 1300 50  0001 C CNN
 	1    8800 1300
@@
 F 0 "R13" V 8996 1000 50  0000 C CNN
 F 1 "49.9" V 8905 1000 50  0000 C CNN
-F 2 "" H 8800 1000 50  0001 C CNN
+F 2 "Resistor_SMD:R_0603_1608Metric" H 8800 1000 50  0001 C CNN
 F 3 "~" H 8800 1000 50  0001 C CNN
 	1    8800 1000
@@
 F 0 "C15" V 9029 2250 50  0000 C CNN
 F 1 "0.1u" V 8938 2250 50  0000 C CNN
-F 2 "" H 8800 2250 50  0001 C CNN
+F 2 "Capacitor_SMD:C_0603_1608Metric" H 8800 2250 50  0001 C CNN
 F 3 "~" H 8800 2250 50  0001 C CNN
 	1    8800 2250
@@
 F 0 "C16" V 9029 2600 50  0000 C CNN
 F 1 "0.1u" V 8938 2600 50  0000 C CNN
-F 2 "" H 8800 2600 50  0001 C CNN
+F 2 "Capacitor_SMD:C_0603_1608Metric" H 8800 2600 50  0001 C CNN
 F 3 "~" H 8800 2600 50  0001 C CNN
 	1    8800 2600
@@
 F 0 "SW1" V 7996 3198 50  0000 L CNN
 F 1 "RST_SW" V 7905 3198 50  0000 L CNN
-F 2 "" H 7950 3250 50  0001 C CNN
+F 2 "Button_Switch_SMD:SW_SPST_B3S-1000" H 7950 3250 50  0001 C CNN
 F 3 "~" H 7950 3250 50  0001 C CNN
 	1    7950 3050
@@
 F 0 "R18" V 7554 2750 50  0000 C CNN
 F 1 "100" V 7645 2750 50  0000 C CNN
-F 2 "" H 7750 2750 50  0001 C CNN
+F 2 "Resistor_SMD:R_0603_1608Metric" H 7750 2750 50  0001 C CNN
 F 3 "~" H 7750 2750 50  0001 C CNN
 	1    7750 2750
@@
 F 0 "C17" H 7358 2996 50  0000 R CNN
 F 1 "0.1u" H 7358 2905 50  0000 R CNN
-F 2 "" H 7450 2950 50  0001 C CNN
+F 2 "Capacitor_SMD:C_0603_1608Metric" H 7450 2950 50  0001 C CNN
 F 3 "~" H 7450 2950 50  0001 C CNN
 	1    7450 2950
@@
 F 0 "R17" H 7441 2504 50  0000 R CNN
 F 1 "10k" H 7441 2595 50  0000 R CNN
-F 2 "" H 7500 2550 50  0001 C CNN
+F 2 "Resistor_SMD:R_0603_1608Metric" H 7500 2550 50  0001 C CNN
 F 3 "~" H 7500 2550 50  0001 C CNN
 	1    7500 2550
@@
 Wire Wire Line
 	5600 1250 5600 1300
-Wire Bus Line
-	1700 4850 1700 7600
-Wire Bus Line
-	6000 2200 6000 7600
 $Comp
 L power:GND #PWR0145
@@
 	1    0    0    -1
 $EndComp
+Wire Bus Line
+	1700 4850 1700 7600
+Wire Bus Line
+	6000 2200 6000 7600
 $EndSCHEMATC

Commit message: added rtc battery footprint
Parts:
- BT1: footprint (none) -> Battery:BatteryHolder_Keystone_1058_1x2032
Changed lines of the file:
@@
 F 0 "BT1" H 1568 1396 50  0000 L CNN
 F 1 "Battery_Cell" H 1568 1305 50  0000 L CNN
-F 2 "" V 1450 1360 50  0001 C CNN
+F 2 "Battery:BatteryHolder_Keystone_1058_1x2032" V 1450 1360 50  0001 C CNN
 F 3 "~" V 1450 1360 50  0001 C CNN
 	1    1450 1300

Commit message: regenerated netlist/annotations and refdeses. using new connector symbol.
Parts:
- renumbered BT1 to BT401, C3 to C401, C4 to C402, C2 to C403, C5 to C404, C6 to C405, C7 to C406, C8 to C407, C9 to C408, C10 to C409, C13 to C410, C12 to C411, C11 to C412, C17 to C413, C15 to C414, C16 to C415, C1 to C416, D1 to D401, D2 to D402, D3 to D403, D4 to D404, D5 to D405, D6 to D406, D7 to D407, R6 to R401, R3 to R402, R1 to R403, R2 to R404, R17 to R405, R18 to R406, R5 to R407, R7 to R408, R13 to R409, R14 to R410, R15 to R411, R16 to R412, R8 to R413, R9 to R414, R10 to R415, R11 to R416, R12 to R417, SW1 to SW401, U1 to U401, Y1 to Y401, Y2 to Y402

Commit message: started layout. fixing some netnames.
Connections:
- net labels added: USER_LED1_CATHODE, USER_LED2_CATHODE, USER_LED3_CATHODE
- net labels removed: USER_LED1_CATHOD
- wire segments 248 -> 249
Changed lines of the file:
@@
 	2750 2850 2450 2850
-Wire Wire Line
-	2450 2850 2450 2600
 Wire Wire Line
 	2450 2550 2750 2550
@@
 	10150 2550 10150 2700
 Text Label 9050 5750 0    50   ~ 0
-USER_LED1_CATHOD
+USER_LED2_CATHODE
 Text Label 9050 4450 0    50   ~ 0
 USER_LED0_CATHODE
@@
 $EndComp
 Text Label 10150 5750 0    50   ~ 0
-USER_LED1_CATHOD
+USER_LED3_CATHODE
 Text Label 10150 4450 0    50   ~ 0
-USER_LED0_CATHODE
+USER_LED1_CATHODE
 $Comp
 L Device:R_Small R412
@@
 	1800 2600 2450 2600
 Connection ~ 1800 2600
-Connection ~ 2450 2600
-Wire Wire Line
-	2450 2600 2450 2550
 Wire Wire Line
 	1450 2350 1600 2350
@@
 	1    0    0    -1
 $EndComp
+Wire Wire Line
+	2450 2600 2600 2600
+Wire Wire Line
+	2600 2600 2600 2650
 Wire Bus Line
 	1700 4850 1700 7600
 Wire Bus Line
 	6000 2200 6000 7600
+Connection ~ 2600 2650
+Wire Wire Line
+	2450 2550 2450 2850
 $EndSCHEMATC
