File: USB_to_UART.sch (KiCad schematic (older format))
At the start: 7 parts

Commit message: Fixed some componenet values. Added some layout notes. added decoupling cap to usb-to-uart circuit.
Parts:
- added C20: 0.1u, symbol Device:C_Small
- gave numbers to parts that had none: 7
Connections:
- wire segments 39 -> 43
Changed lines of the file:
@@
 P 6750 3250
 AR Path="/5D6F460E" Ref="U?"  Part="1"
-AR Path="/5D6EF68B/5D6F460E" Ref="U?"  Part="1"
-F 0 "U?" H 6750 4431 50  0000 C CNN
+AR Path="/5D6EF68B/5D6F460E" Ref="U4"  Part="1"
+F 0 "U4" H 6750 4431 50  0000 C CNN
 F 1 "FT232RL" H 6750 4340 50  0000 C CNN
 F 2 "Package_SO:SSOP-28_5.3x10.2mm_P0.65mm" H 6750 3250 50  0001 C CNN
@@
 Wire Wire Line
 	6650 2250 6650 2000
-Wire Wire Line
-	6850 2250 6850 2000
 $Comp
 L Connector:USB_B_Micro J?
@@
 P 8400 2850
 AR Path="/5D6F4616" Ref="J?"  Part="1"
-AR Path="/5D6EF68B/5D6F4616" Ref="J?"  Part="1"
-F 0 "J?" H 8457 3317 50  0000 C CNN
+AR Path="/5D6EF68B/5D6F4616" Ref="J1"  Part="1"
+F 0 "J1" H 8457 3317 50  0000 C CNN
 F 1 "USB_B_Micro" H 8457 3226 50  0000 C CNN
 F 2 "" H 8550 2800 50  0001 C CNN
@@
 P 7800 3100
 AR Path="/5D6F461C" Ref="R?"  Part="1"
-AR Path="/5D6EF68B/5D6F461C" Ref="R?"  Part="1"
-F 0 "R?" H 7859 3146 50  0000 L CNN
+AR Path="/5D6EF68B/5D6F461C" Ref="R19"  Part="1"
+F 0 "R19" H 7859 3146 50  0000 L CNN
 F 1 "4.7k" H 7859 3055 50  0000 L CNN
 F 2 "" H 7800 3100 50  0001 C CNN
@@
 P 7800 3400
 AR Path="/5D6F4622" Ref="R?"  Part="1"
-AR Path="/5D6EF68B/5D6F4622" Ref="R?"  Part="1"
-F 0 "R?" H 7859 3446 50  0000 L CNN
+AR Path="/5D6EF68B/5D6F4622" Ref="R20"  Part="1"
+F 0 "R20" H 7859 3446 50  0000 L CNN
 F 1 "10k" H 7859 3355 50  0000 L CNN
 F 2 "" H 7800 3400 50  0001 C CNN
@@
 P 7800 3550
 AR Path="/5D6F462B" Ref="#PWR?"  Part="1"
-AR Path="/5D6EF68B/5D6F462B" Ref="#PWR?"  Part="1"
-F 0 "#PWR?" H 7800 3300 50  0001 C CNN
+AR Path="/5D6EF68B/5D6F462B" Ref="#PWR0135"  Part="1"
+F 0 "#PWR0135" H 7800 3300 50  0001 C CNN
 F 1 "GND" H 7805 3377 50  0000 C CNN
 F 2 "" H 7800 3550 50  0001 C CNN
@@
 P 7700 2550
 AR Path="/5D6F4632" Ref="C?"  Part="1"
-AR Path="/5D6EF68B/5D6F4632" Ref="C?"  Part="1"
-F 0 "C?" V 7471 2550 50  0000 C CNN
+AR Path="/5D6EF68B/5D6F4632" Ref="C18"  Part="1"
+F 0 "C18" V 7471 2550 50  0000 C CNN
 F 1 "100nF" V 7562 2550 50  0000 C CNN
 F 2 "" H 7700 2550 50  0001 C CNN
@@
 P 7850 2550
 AR Path="/5D6F4638" Ref="#PWR?"  Part="1"
-AR Path="/5D6EF68B/5D6F4638" Ref="#PWR?"  Part="1"
-F 0 "#PWR?" H 7850 2300 50  0001 C CNN
+AR Path="/5D6EF68B/5D6F4638" Ref="#PWR0136"  Part="1"
+F 0 "#PWR0136" H 7850 2300 50  0001 C CNN
 F 1 "GND" V 7855 2422 50  0000 R CNN
 F 2 "" H 7850 2550 50  0001 C CNN
@@
 P 8000 3150
 AR Path="/5D6F4645" Ref="#PWR?"  Part="1"
-AR Path="/5D6EF68B/5D6F4645" Ref="#PWR?"  Part="1"
-F 0 "#PWR?" H 8000 2900 50  0001 C CNN
+AR Path="/5D6EF68B/5D6F4645" Ref="#PWR0137"  Part="1"
+F 0 "#PWR0137" H 8000 2900 50  0001 C CNN
 F 1 "GND" H 8005 2977 50  0000 C CNN
 F 2 "" H 8000 3150 50  0001 C CNN
@@
 P 6750 4400
 AR Path="/5D6F4654" Ref="#PWR?"  Part="1"
-AR Path="/5D6EF68B/5D6F4654" Ref="#PWR?"  Part="1"
-F 0 "#PWR?" H 6750 4150 50  0001 C CNN
+AR Path="/5D6EF68B/5D6F4654" Ref="#PWR0138"  Part="1"
+F 0 "#PWR0138" H 6750 4150 50  0001 C CNN
 F 1 "GND" H 6755 4227 50  0000 C CNN
 F 2 "" H 6750 4400 50  0001 C CNN
@@
 P 8400 3950
 AR Path="/5D6F465D" Ref="#PWR?"  Part="1"
-AR Path="/5D6EF68B/5D6F465D" Ref="#PWR?"  Part="1"
-F 0 "#PWR?" H 8400 3700 50  0001 C CNN
+AR Path="/5D6EF68B/5D6F465D" Ref="#PWR0139"  Part="1"
+F 0 "#PWR0139" H 8400 3700 50  0001 C CNN
 F 1 "GND" H 8405 3777 50  0000 C CNN
 F 2 "" H 8400 3950 50  0001 C CNN
@@
 P 7650 4100
 AR Path="/5D6F4665" Ref="#PWR?"  Part="1"
-AR Path="/5D6EF68B/5D6F4665" Ref="#PWR?"  Part="1"
-F 0 "#PWR?" H 7650 3850 50  0001 C CNN
+AR Path="/5D6EF68B/5D6F4665" Ref="#PWR0140"  Part="1"
+F 0 "#PWR0140" H 7650 3850 50  0001 C CNN
 F 1 "GND" H 7655 3927 50  0000 C CNN
 F 2 "" H 7650 4100 50  0001 C CNN
@@
 P 8300 3700
 AR Path="/5D6F466D" Ref="C?"  Part="1"
-AR Path="/5D6EF68B/5D6F466D" Ref="C?"  Part="1"
-F 0 "C?" H 8000 3700 50  0000 L CNN
+AR Path="/5D6EF68B/5D6F466D" Ref="C19"  Part="1"
+F 0 "C19" H 8000 3700 50  0000 L CNN
 F 1 "3300pF" H 8000 3600 50  0000 L CNN
 F 2 "" H 8338 3550 50  0001 C CNN
@@
 P 8550 3700
 AR Path="/5D6F4673" Ref="R?"  Part="1"
-AR Path="/5D6EF68B/5D6F4673" Ref="R?"  Part="1"
-F 0 "R?" H 8620 3746 50  0000 L CNN
+AR Path="/5D6EF68B/5D6F4673" Ref="R21"  Part="1"
+F 0 "R21" H 8620 3746 50  0000 L CNN
 F 1 "1M" H 8620 3655 50  0000 L CNN
 F 2 "" V 8480 3700 50  0001 C CNN
@@
 P 8500 3300
 AR Path="/5D6F4685" Ref="#PWR?"  Part="1"
-AR Path="/5D6EF68B/5D6F4685" Ref="#PWR?"  Part="1"
-F 0 "#PWR?" H 8500 3050 50  0001 C CNN
+AR Path="/5D6EF68B/5D6F4685" Ref="#PWR0141"  Part="1"
+F 0 "#PWR0141" H 8500 3050 50  0001 C CNN
 F 1 "GND" H 8600 3200 50  0000 C CNN
 F 2 "" H 8500 3300 50  0001 C CNN
@@
 P 6850 2000
 AR Path="/5D6F5C8E" Ref="#PWR?"  Part="1"
-AR Path="/5D6EF68B/5D6F5C8E" Ref="#PWR?"  Part="1"
-F 0 "#PWR?" H 6850 1850 50  0001 C CNN
+AR Path="/5D6EF68B/5D6F5C8E" Ref="#PWR0142"  Part="1"
+F 0 "#PWR0142" H 6850 1850 50  0001 C CNN
 F 1 "+3.3V" H 6865 2173 50  0000 C CNN
 F 2 "" H 6850 2000 50  0001 C CNN
@@
 P 6650 2000
 AR Path="/5D6F5C94" Ref="#PWR?"  Part="1"
-AR Path="/5D6EF68B/5D6F5C94" Ref="#PWR?"  Part="1"
-F 0 "#PWR?" H 6650 1850 50  0001 C CNN
+AR Path="/5D6EF68B/5D6F5C94" Ref="#PWR0143"  Part="1"
+F 0 "#PWR0143" H 6650 1850 50  0001 C CNN
 F 1 "+5V" H 6665 2173 50  0000 C CNN
 F 2 "" H 6650 2000 50  0001 C CNN
@@
 Text HLabel 5700 2850 0    50   Input ~ 0
 UART_CTS
+$Comp
+L Device:C_Small C20
+U 1 1 5D18887F
+P 7050 2100
+F 0 "C20" V 6821 2100 50  0000 C CNN
+F 1 "0.1u" V 6912 2100 50  0000 C CNN
+F 2 "" H 7050 2100 50  0001 C CNN
+F 3 "~" H 7050 2100 50  0001 C CNN
+	1    7050 2100
+	0    1    1    0
+$EndComp
+Wire Wire Line
+	7150 2100 7250 2100
+Wire Wire Line
+	7250 2100 7250 2150
+$Comp
+L power:GND #PWR0146
+U 1 1 5D18A53E
+P 7250 2150
+F 0 "#PWR0146" H 7250 1900 50  0001 C CNN
+F 1 "GND" H 7255 1977 50  0000 C CNN
+F 2 "" H 7250 2150 50  0001 C CNN
+F 3 "" H 7250 2150 50  0001 C CNN
+	1    7250 2150
+	1    0    0    -1
+$EndComp
+Wire Wire Line
+	6850 2000 6850 2100
+Wire Wire Line
+	6950 2100 6850 2100
+Connection ~ 6850 2100
+Wire Wire Line
+	6850 2100 6850 2250
 $EndSCHEMATC

Commit message: added part footprints. added usb-uart leds.
Parts:
- added D8, D9: LED, Diode_SMD:D_0805_2012Metric, symbol Device:LED
- added R25, R26: 330, Resistor_SMD:R_0603_1608Metric, symbol Device:R_Small
- C18, C19, C20: footprint (none) -> Capacitor_SMD:C_0603_1608Metric
- J1: footprint (none) -> Connector_USB:USB_Micro-B_Molex-105017-0001
- R19, R20, R21: footprint (none) -> Resistor_SMD:R_0603_1608Metric
Connections:
- net labels added: USB_LED_0, USB_LED_1
- wire segments 43 -> 51
Changed lines of the file:
@@
 F 0 "J1" H 8457 3317 50  0000 C CNN
 F 1 "USB_B_Micro" H 8457 3226 50  0000 C CNN
-F 2 "" H 8550 2800 50  0001 C CNN
+F 2 "Connector_USB:USB_Micro-B_Molex-105017-0001" H 8550 2800 50  0001 C CNN
 F 3 "~" H 8550 2800 50  0001 C CNN
 	1    8400 2850
@@
 F 0 "R19" H 7859 3146 50  0000 L CNN
 F 1 "4.7k" H 7859 3055 50  0000 L CNN
-F 2 "" H 7800 3100 50  0001 C CNN
+F 2 "Resistor_SMD:R_0603_1608Metric" H 7800 3100 50  0001 C CNN
 F 3 "~" H 7800 3100 50  0001 C CNN
 	1    7800 3100
@@
 F 0 "R20" H 7859 3446 50  0000 L CNN
 F 1 "10k" H 7859 3355 50  0000 L CNN
-F 2 "" H 7800 3400 50  0001 C CNN
+F 2 "Resistor_SMD:R_0603_1608Metric" H 7800 3400 50  0001 C CNN
 F 3 "~" H 7800 3400 50  0001 C CNN
 	1    7800 3400
@@
 F 0 "C18" V 7471 2550 50  0000 C CNN
 F 1 "100nF" V 7562 2550 50  0000 C CNN
-F 2 "" H 7700 2550 50  0001 C CNN
+F 2 "Capacitor_SMD:C_0603_1608Metric" H 7700 2550 50  0001 C CNN
 F 3 "~" H 7700 2550 50  0001 C CNN
 	1    7700 2550
@@
 F 0 "C19" H 8000 3700 50  0000 L CNN
 F 1 "3300pF" H 8000 3600 50  0000 L CNN
-F 2 "" H 8338 3550 50  0001 C CNN
+F 2 "Capacitor_SMD:C_0603_1608Metric" H 8338 3550 50  0001 C CNN
 F 3 "~" H 8300 3700 50  0001 C CNN
 	1    8300 3700
@@
 F 0 "R21" H 8620 3746 50  0000 L CNN
 F 1 "1M" H 8620 3655 50  0000 L CNN
-F 2 "" V 8480 3700 50  0001 C CNN
+F 2 "Resistor_SMD:R_0603_1608Metric" V 8480 3700 50  0001 C CNN
 F 3 "~" H 8550 3700 50  0001 C CNN
 	1    8550 3700
@@
 F 0 "C20" V 6821 2100 50  0000 C CNN
 F 1 "0.1u" V 6912 2100 50  0000 C CNN
-F 2 "" H 7050 2100 50  0001 C CNN
+F 2 "Capacitor_SMD:C_0603_1608Metric" H 7050 2100 50  0001 C CNN
 F 3 "~" H 7050 2100 50  0001 C CNN
 	1    7050 2100
@@
 Wire Wire Line
 	6850 2100 6850 2250
+Wire Wire Line
+	5700 3650 5700 3700
+$Comp
+L Device:R_Small R25
+U 1 1 5D17BA3C
+P 5350 4200
+F 0 "R25" H 5409 4246 50  0000 L CNN
+F 1 "330" H 5409 4155 50  0000 L CNN
+F 2 "Resistor_SMD:R_0603_1608Metric" H 5350 4200 50  0001 C CNN
+F 3 "~" H 5350 4200 50  0001 C CNN
+	1    5350 4200
+	1    0    0    -1
+$EndComp
+$Comp
+L Device:R_Small R26
+U 1 1 5D17BCA6
+P 5700 4200
+F 0 "R26" H 5759 4246 50  0000 L CNN
+F 1 "330" H 5759 4155 50  0000 L CNN
+F 2 "Resistor_SMD:R_0603_1608Metric" H 5700 4200 50  0001 C CNN
+F 3 "~" H 5700 4200 50  0001 C CNN
+	1    5700 4200
+	1    0    0    -1
+$EndComp
+$Comp
+L power:GND #PWR01
+U 1 1 5D17C3F5
+P 5350 4350
+F 0 "#PWR01" H 5350 4100 50  0001 C CNN
+F 1 "GND" H 5355 4177 50  0000 C CNN
+F 2 "" H 5350 4350 50  0001 C CNN
+F 3 "" H 5350 4350 50  0001 C CNN
+	1    5350 4350
+	1    0    0    -1
+$EndComp
+$Comp
+L power:GND #PWR02
+U 1 1 5D17C5C9
+P 5700 4350
+F 0 "#PWR02" H 5700 4100 50  0001 C CNN
+F 1 "GND" H 5705 4177 50  0000 C CNN
+F 2 "" H 5700 4350 50  0001 C CNN
+F 3 "" H 5700 4350 50  0001 C CNN
+	1    5700 4350
+	1    0    0    -1
+$EndComp
+Wire Wire Line
+	5700 4350 5700 4300
+Wire Wire Line
+	5350 4300 5350 4350
+$Comp
+L Device:LED D8
+U 1 1 5D1932B7
+P 5350 3850
+F 0 "D8" V 5389 3733 50  0000 R CNN
+F 1 "LED" V 5298 3733 50  0000 R CNN
+F 2 "Diode_SMD:D_0805_2012Metric" H 5350 3850 50  0001 C CNN
+F 3 "~" H 5350 3850 50  0001 C CNN
+	1    5350 3850
+	0    -1   -1   0
+$EndComp
+Wire Wire Line
+	5350 3550 5350 3700
+Wire Wire Line
+	5350 4100 5350 4000
+$Comp
+L Device:LED D9
+U 1 1 5D19C25D
+P 5700 3850
+F 0 "D9" V 5739 3733 50  0000 R CNN
+F 1 "LED" V 5648 3733 50  0000 R CNN
+F 2 "Diode_SMD:D_0805_2012Metric" H 5700 3850 50  0001 C CNN
+F 3 "~" H 5700 3850 50  0001 C CNN
+	1    5700 3850
+	0    -1   -1   0
+$EndComp
+Wire Wire Line
+	5700 4100 5700 4000
+Wire Wire Line
+	5700 3650 5950 3650
+Wire Wire Line
+	5350 3550 5950 3550
+Text Label 5350 3550 0    50   ~ 0
+USB_LED_0
+Text Label 5950 3650 2    50   ~ 0
+USB_LED_1
 $EndSCHEMATC

Commit message: regenerated netlist/annotations and refdeses. using new connector symbol.
Parts:
- renumbered C20 to C501, C18 to C502, C19 to C503, D8 to D501, D9 to D502, J1 to J501, R25 to R501, R26 to R502, R19 to R503, R20 to R504, R21 to R505, U4 to U501
Changed lines of the file:
@@
 P 6750 3250
 AR Path="/5D6F460E" Ref="U?"  Part="1"
-AR Path="/5D6EF68B/5D6F460E" Ref="U4"  Part="1"
-F 0 "U4" H 6750 4431 50  0000 C CNN
+AR Path="/5D6EF68B/5D6F460E" Ref="U501"  Part="1"
+F 0 "U501" H 6750 4431 50  0000 C CNN
 F 1 "FT232RL" H 6750 4340 50  0000 C CNN
 F 2 "Package_SO:SSOP-28_5.3x10.2mm_P0.65mm" H 6750 3250 50  0001 C CNN
@@
 P 8400 2850
 AR Path="/5D6F4616" Ref="J?"  Part="1"
-AR Path="/5D6EF68B/5D6F4616" Ref="J1"  Part="1"
-F 0 "J1" H 8457 3317 50  0000 C CNN
+AR Path="/5D6EF68B/5D6F4616" Ref="J501"  Part="1"
+F 0 "J501" H 8457 3317 50  0000 C CNN
 F 1 "USB_B_Micro" H 8457 3226 50  0000 C CNN
 F 2 "Connector_USB:USB_Micro-B_Molex-105017-0001" H 8550 2800 50  0001 C CNN
@@
 P 7800 3100
 AR Path="/5D6F461C" Ref="R?"  Part="1"
-AR Path="/5D6EF68B/5D6F461C" Ref="R19"  Part="1"
-F 0 "R19" H 7859 3146 50  0000 L CNN
+AR Path="/5D6EF68B/5D6F461C" Ref="R503"  Part="1"
+F 0 "R503" H 7859 3146 50  0000 L CNN
 F 1 "4.7k" H 7859 3055 50  0000 L CNN
 F 2 "Resistor_SMD:R_0603_1608Metric" H 7800 3100 50  0001 C CNN
@@
 P 7800 3400
 AR Path="/5D6F4622" Ref="R?"  Part="1"
-AR Path="/5D6EF68B/5D6F4622" Ref="R20"  Part="1"
-F 0 "R20" H 7859 3446 50  0000 L CNN
+AR Path="/5D6EF68B/5D6F4622" Ref="R504"  Part="1"
+F 0 "R504" H 7859 3446 50  0000 L CNN
 F 1 "10k" H 7859 3355 50  0000 L CNN
 F 2 "Resistor_SMD:R_0603_1608Metric" H 7800 3400 50  0001 C CNN
@@
 P 7800 3550
 AR Path="/5D6F462B" Ref="#PWR?"  Part="1"
-AR Path="/5D6EF68B/5D6F462B" Ref="#PWR0135"  Part="1"
-F 0 "#PWR0135" H 7800 3300 50  0001 C CNN
+AR Path="/5D6EF68B/5D6F462B" Ref="#PWR0508"  Part="1"
+F 0 "#PWR0508" H 7800 3300 50  0001 C CNN
 F 1 "GND" H 7805 3377 50  0000 C CNN
 F 2 "" H 7800 3550 50  0001 C CNN
@@
 P 7700 2550
 AR Path="/5D6F4632" Ref="C?"  Part="1"
-AR Path="/5D6EF68B/5D6F4632" Ref="C18"  Part="1"
-F 0 "C18" V 7471 2550 50  0000 C CNN
+AR Path="/5D6EF68B/5D6F4632" Ref="C502"  Part="1"
+F 0 "C502" V 7471 2550 50  0000 C CNN
 F 1 "100nF" V 7562 2550 50  0000 C CNN
 F 2 "Capacitor_SMD:C_0603_1608Metric" H 7700 2550 50  0001 C CNN
@@
 P 7850 2550
 AR Path="/5D6F4638" Ref="#PWR?"  Part="1"
-AR Path="/5D6EF68B/5D6F4638" Ref="#PWR0136"  Part="1"
-F 0 "#PWR0136" H 7850 2300 50  0001 C CNN
+AR Path="/5D6EF68B/5D6F4638" Ref="#PWR0509"  Part="1"
+F 0 "#PWR0509" H 7850 2300 50  0001 C CNN
 F 1 "GND" V 7855 2422 50  0000 R CNN
 F 2 "" H 7850 2550 50  0001 C CNN
@@
 P 8000 3150
 AR Path="/5D6F4645" Ref="#PWR?"  Part="1"
-AR Path="/5D6EF68B/5D6F4645" Ref="#PWR0137"  Part="1"
-F 0 "#PWR0137" H 8000 2900 50  0001 C CNN
+AR Path="/5D6EF68B/5D6F4645" Ref="#PWR0510"  Part="1"
+F 0 "#PWR0510" H 8000 2900 50  0001 C CNN
 F 1 "GND" H 8005 2977 50  0000 C CNN
 F 2 "" H 8000 3150 50  0001 C CNN
@@
 P 6750 4400
 AR Path="/5D6F4654" Ref="#PWR?"  Part="1"
-AR Path="/5D6EF68B/5D6F4654" Ref="#PWR0138"  Part="1"
-F 0 "#PWR0138" H 6750 4150 50  0001 C CNN
+AR Path="/5D6EF68B/5D6F4654" Ref="#PWR0504"  Part="1"
+F 0 "#PWR0504" H 6750 4150 50  0001 C CNN
 F 1 "GND" H 6755 4227 50  0000 C CNN
 F 2 "" H 6750 4400 50  0001 C CNN
@@
 P 8400 3950
 AR Path="/5D6F465D" Ref="#PWR?"  Part="1"
-AR Path="/5D6EF68B/5D6F465D" Ref="#PWR0139"  Part="1"
-F 0 "#PWR0139" H 8400 3700 50  0001 C CNN
+AR Path="/5D6EF68B/5D6F465D" Ref="#PWR0511"  Part="1"
+F 0 "#PWR0511" H 8400 3700 50  0001 C CNN
 F 1 "GND" H 8405 3777 50  0000 C CNN
 F 2 "" H 8400 3950 50  0001 C CNN
@@
 P 7650 4100
 AR Path="/5D6F4665" Ref="#PWR?"  Part="1"
-AR Path="/5D6EF68B/5D6F4665" Ref="#PWR0140"  Part="1"
-F 0 "#PWR0140" H 7650 3850 50  0001 C CNN
+AR Path="/5D6EF68B/5D6F4665" Ref="#PWR0507"  Part="1"
+F 0 "#PWR0507" H 7650 3850 50  0001 C CNN
 F 1 "GND" H 7655 3927 50  0000 C CNN
 F 2 "" H 7650 4100 50  0001 C CNN
@@
 P 8300 3700
 AR Path="/5D6F466D" Ref="C?"  Part="1"
-AR Path="/5D6EF68B/5D6F466D" Ref="C19"  Part="1"
-F 0 "C19" H 8000 3700 50  0000 L CNN
+AR Path="/5D6EF68B/5D6F466D" Ref="C503"  Part="1"
+F 0 "C503" H 8000 3700 50  0000 L CNN
 F 1 "3300pF" H 8000 3600 50  0000 L CNN
 F 2 "Capacitor_SMD:C_0603_1608Metric" H 8338 3550 50  0001 C CNN
@@
 P 8550 3700
 AR Path="/5D6F4673" Ref="R?"  Part="1"
-AR Path="/5D6EF68B/5D6F4673" Ref="R21"  Part="1"
-F 0 "R21" H 8620 3746 50  0000 L CNN
+AR Path="/5D6EF68B/5D6F4673" Ref="R505"  Part="1"
+F 0 "R505" H 8620 3746 50  0000 L CNN
 F 1 "1M" H 8620 3655 50  0000 L CNN
 F 2 "Resistor_SMD:R_0603_1608Metric" V 8480 3700 50  0001 C CNN
@@
 P 8500 3300
 AR Path="/5D6F4685" Ref="#PWR?"  Part="1"
-AR Path="/5D6EF68B/5D6F4685" Ref="#PWR0141"  Part="1"
-F 0 "#PWR0141" H 8500 3050 50  0001 C CNN
+AR Path="/5D6EF68B/5D6F4685" Ref="#PWR0512"  Part="1"
+F 0 "#PWR0512" H 8500 3050 50  0001 C CNN
 F 1 "GND" H 8600 3200 50  0000 C CNN
 F 2 "" H 8500 3300 50  0001 C CNN
@@
 P 6850 2000
 AR Path="/5D6F5C8E" Ref="#PWR?"  Part="1"
-AR Path="/5D6EF68B/5D6F5C8E" Ref="#PWR0142"  Part="1"
-F 0 "#PWR0142" H 6850 1850 50  0001 C CNN
+AR Path="/5D6EF68B/5D6F5C8E" Ref="#PWR0505"  Part="1"
+F 0 "#PWR0505" H 6850 1850 50  0001 C CNN
 F 1 "+3.3V" H 6865 2173 50  0000 C CNN
 F 2 "" H 6850 2000 50  0001 C CNN
@@
 P 6650 2000
 AR Path="/5D6F5C94" Ref="#PWR?"  Part="1"
-AR Path="/5D6EF68B/5D6F5C94" Ref="#PWR0143"  Part="1"
-F 0 "#PWR0143" H 6650 1850 50  0001 C CNN
+AR Path="/5D6EF68B/5D6F5C94" Ref="#PWR0503"  Part="1"
+F 0 "#PWR0503" H 6650 1850 50  0001 C CNN
 F 1 "+5V" H 6665 2173 50  0000 C CNN
 F 2 "" H 6650 2000 50  0001 C CNN
@@
 UART_CTS
 $Comp
-L Device:C_Small C20
+L Device:C_Small C501
 U 1 1 5D18887F
 P 7050 2100
-F 0 "C20" V 6821 2100 50  0000 C CNN
+F 0 "C501" V 6821 2100 50  0000 C CNN
 F 1 "0.1u" V 6912 2100 50  0000 C CNN
 F 2 "Capacitor_SMD:C_0603_1608Metric" H 7050 2100 50  0001 C CNN
@@
 	7250 2100 7250 2150
 $Comp
-L power:GND #PWR0146
+L power:GND #PWR0506
 U 1 1 5D18A53E
 P 7250 2150
-F 0 "#PWR0146" H 7250 1900 50  0001 C CNN
+F 0 "#PWR0506" H 7250 1900 50  0001 C CNN
 F 1 "GND" H 7255 1977 50  0000 C CNN
 F 2 "" H 7250 2150 50  0001 C CNN
@@
 	5700 3650 5700 3700
 $Comp
-L Device:R_Small R25
+L Device:R_Small R501
 U 1 1 5D17BA3C
 P 5350 4200
-F 0 "R25" H 5409 4246 50  0000 L CNN
+F 0 "R501" H 5409 4246 50  0000 L CNN
 F 1 "330" H 5409 4155 50  0000 L CNN
 F 2 "Resistor_SMD:R_0603_1608Metric" H 5350 4200 50  0001 C CNN
@@
 $EndComp
 $Comp
-L Device:R_Small R26
+L Device:R_Small R502
 U 1 1 5D17BCA6
 P 5700 4200
-F 0 "R26" H 5759 4246 50  0000 L CNN
+F 0 "R502" H 5759 4246 50  0000 L CNN
 F 1 "330" H 5759 4155 50  0000 L CNN
 F 2 "Resistor_SMD:R_0603_1608Metric" H 5700 4200 50  0001 C CNN
@@
 $EndComp
 $Comp
-L power:GND #PWR01
+L power:GND #PWR0501
 U 1 1 5D17C3F5
 P 5350 4350
-F 0 "#PWR01" H 5350 4100 50  0001 C CNN
+F 0 "#PWR0501" H 5350 4100 50  0001 C CNN
 F 1 "GND" H 5355 4177 50  0000 C CNN
 F 2 "" H 5350 4350 50  0001 C CNN
@@
 $EndComp
 $Comp
-L power:GND #PWR02
+L power:GND #PWR0502
 U 1 1 5D17C5C9
 P 5700 4350
-F 0 "#PWR02" H 5700 4100 50  0001 C CNN
+F 0 "#PWR0502" H 5700 4100 50  0001 C CNN
 F 1 "GND" H 5705 4177 50  0000 C CNN
 F 2 "" H 5700 4350 50  0001 C CNN
@@
 	5350 4300 5350 4350
 $Comp
-L Device:LED D8
+L Device:LED D501
 U 1 1 5D1932B7
 P 5350 3850
-F 0 "D8" V 5389 3733 50  0000 R CNN
+F 0 "D501" V 5389 3733 50  0000 R CNN
 F 1 "LED" V 5298 3733 50  0000 R CNN
 F 2 "Diode_SMD:D_0805_2012Metric" H 5350 3850 50  0001 C CNN
@@
 	5350 4100 5350 4000
 $Comp
-L Device:LED D9
+L Device:LED D502
 U 1 1 5D19C25D
 P 5700 3850
-F 0 "D9" V 5739 3733 50  0000 R CNN
+F 0 "D502" V 5739 3733 50  0000 R CNN
 F 1 "LED" V 5648 3733 50  0000 R CNN
 F 2 "Diode_SMD:D_0805_2012Metric" H 5700 3850 50  0001 C CNN

Commit message: started layout. fixing some netnames.
Connections:
- net labels added: DBG_USB_D_N, DBG_USB_D_P, DBG_USB_SHIELD, DBG_VBUS
Changed lines of the file:
@@
 Text Label 5950 3650 2    50   ~ 0
 USB_LED_1
+Text Label 7600 2850 0    50   ~ 0
+DBG_USB_D_P
+Text Label 7600 2950 0    50   ~ 0
+DBG_USB_D_N
+Text Label 7800 2650 0    50   ~ 0
+DBG_VBUS
+Text Label 8450 3500 0    50   ~ 0
+DBG_USB_SHIELD
 $EndSCHEMATC

Commit message: sourced all parts, except LEDs. added bom. fixed a few footprints/values.
Parts:
- D501, D502: footprint Diode_SMD:D_0805_2012Metric -> LED_SMD:LED_0805_2012Metric
Changed lines of the file:
@@
 $Descr A4 11693 8268
 encoding utf-8
-Sheet 5 6
+Sheet 6 6
 Title ""
 Date ""
@@
 F 0 "D501" V 5389 3733 50  0000 R CNN
 F 1 "LED" V 5298 3733 50  0000 R CNN
-F 2 "Diode_SMD:D_0805_2012Metric" H 5350 3850 50  0001 C CNN
+F 2 "LED_SMD:LED_0805_2012Metric" H 5350 3850 50  0001 C CNN
 F 3 "~" H 5350 3850 50  0001 C CNN
 	1    5350 3850
@@
 F 0 "D502" V 5739 3733 50  0000 R CNN
 F 1 "LED" V 5648 3733 50  0000 R CNN
-F 2 "Diode_SMD:D_0805_2012Metric" H 5700 3850 50  0001 C CNN
+F 2 "LED_SMD:LED_0805_2012Metric" H 5700 3850 50  0001 C CNN
 F 3 "~" H 5700 3850 50  0001 C CNN
 	1    5700 3850
