File: v_batt.sch (KiCad schematic (older format))
At the start: 3 parts, among them U1 LT1761-3

Commit message: removed rc filter on vbatt output. Included ltspice sim to prove it's unneeded.
Parts:
- added C3: 1u, Capacitor_SMD:C_0603_1608Metric, symbol Device:C_Small
- C1: value 0.1u -> 0.01u
Connections:
- wire segments 12 -> 15
Changed lines of the file:
@@
 $EndComp
 Wire Wire Line
-	4200 3600 4150 3600
-Wire Wire Line
-	4150 3600 4150 3700
-Wire Wire Line
-	4150 3700 4200 3700
-Wire Wire Line
-	4150 3600 4150 3500
-Connection ~ 4150 3600
+	3850 3600 3850 3500
 $Comp
 L power:+BATT #PWR?
 U 1 1 5D2F3127
-P 4150 3500
+P 3850 3500
 AR Path="/5C80AE96/5D2F3127" Ref="#PWR?"  Part="1"
 AR Path="/5C80AE96/5D2CB049/5D2F3127" Ref="#PWR0101"  Part="1"
-F 0 "#PWR0101" H 4150 3350 50  0001 C CNN
-F 1 "+BATT" H 4165 3673 50  0000 C CNN
-F 2 "" H 4150 3500 50  0001 C CNN
-F 3 "" H 4150 3500 50  0001 C CNN
-	1    4150 3500
+F 0 "#PWR0101" H 3850 3350 50  0001 C CNN
+F 1 "+BATT" H 3865 3673 50  0000 C CNN
+F 2 "" H 3850 3500 50  0001 C CNN
+F 3 "" H 3850 3500 50  0001 C CNN
+	1    3850 3500
 	1    0    0    -1
 $EndComp
 Wire Wire Line
-	4600 4000 4600 4050
+	3950 3800 3950 3850
 $Comp
 L power:GND #PWR?
 U 1 1 5D2F312E
-P 4600 4050
+P 3950 3850
 AR Path="/5C80AE96/5D2F312E" Ref="#PWR?"  Part="1"
 AR Path="/5C80AE96/5D2CB049/5D2F312E" Ref="#PWR0102"  Part="1"
-F 0 "#PWR0102" H 4600 3800 50  0001 C CNN
-F 1 "GND" H 4605 3877 50  0000 C CNN
-F 2 "" H 4600 4050 50  0001 C CNN
-F 3 "" H 4600 4050 50  0001 C CNN
-	1    4600 4050
+F 0 "#PWR0102" H 3950 3600 50  0001 C CNN
+F 1 "GND" H 3955 3677 50  0000 C CNN
+F 2 "" H 3950 3850 50  0001 C CNN
+F 3 "" H 3950 3850 50  0001 C CNN
+	1    3950 3850
 	1    0    0    -1
 $EndComp
@@
 AR Path="/5C80AE96/5D2CB049/5D2F3141" Ref="C1"  Part="1"
 F 0 "C1" H 5242 3746 50  0000 L CNN
-F 1 "0.1u" H 5242 3655 50  0000 L CNN
+F 1 "0.01u" H 5242 3655 50  0000 L CNN
 F 2 "Capacitor_SMD:C_0603_1608Metric" H 5150 3700 50  0001 C CNN
 F 3 "~" H 5150 3700 50  0001 C CNN
@@
 Text HLabel 5700 3600 2    50   Input ~ 0
 Vout
+$Comp
+L Device:C_Small C3
+U 1 1 5D2E6E95
+P 3950 3700
+F 0 "C3" H 4042 3746 50  0000 L CNN
+F 1 "1u" H 4042 3655 50  0000 L CNN
+F 2 "Capacitor_SMD:C_0603_1608Metric" H 3950 3700 50  0001 C CNN
+F 3 "~" H 3950 3700 50  0001 C CNN
+	1    3950 3700
+	1    0    0    -1
+$EndComp
+Wire Wire Line
+	4200 3700 4150 3700
+Wire Wire Line
+	4150 3700 4150 3600
+Wire Wire Line
+	4150 3600 4200 3600
+Wire Wire Line
+	4150 3600 3950 3600
+Connection ~ 4150 3600
+Wire Wire Line
+	3850 3600 3950 3600
+Connection ~ 3950 3600
+$Comp
+L power:GND #PWR?
+U 1 1 5D2E9DCE
+P 4600 4050
+AR Path="/5C80AE96/5D2E9DCE" Ref="#PWR?"  Part="1"
+AR Path="/5C80AE96/5D2CB049/5D2E9DCE" Ref="#PWR0105"  Part="1"
+F 0 "#PWR0105" H 4600 3800 50  0001 C CNN
+F 1 "GND" H 4605 3877 50  0000 C CNN
+F 2 "" H 4600 4050 50  0001 C CNN
+F 3 "" H 4600 4050 50  0001 C CNN
+	1    4600 4050
+	1    0    0    -1
+$EndComp
+Wire Wire Line
+	4600 4050 4600 4000
 $EndSCHEMATC
