File: Raptor2000.kicad_pcb (KiCad board)
At the start: 4 copper layers, 63.5 x 76.2 mm, 80 parts, among them J301 ET60T-000-3-08-D04-x-R1-S-x, J501 USB_B_Micro, SW401 RST_SW, U1 LT1761-3, U201 IS42S16400J-xC, U202 TC58CVG2S0HRAIG, U401 TM4C1294NCPDTGOOD, U501 FT232RL, Y401 Crystal_GND24, Y402 Crystal

Commit message: layout and schematic cleanup.
Parts:
- C201, C202, C203, C204, C205, C206, C207, C409, C416, R404: moved to B.Cu
- moved R405 26.0 mm to (170.9, 87.6), turned to 90 degrees
- moved C409 9.01 mm to (153.3, 84.6), turned to 90 degrees
- moved C416 8.01 mm to (153.3, 81.4), turned to 90 degrees
- moved D502 5.64 mm to (129.3, 63.2), turned to 180 degrees
- moved D501 5.64 mm to (129.3, 60.7), turned to 180 degrees
- moved R502 5.43 mm to (132.8, 63.2)
- moved R504 4.02 mm to (142.7, 61.5), turned to 180 degrees
- moved C502 3.79 mm to (146.1, 61.5), turned to 180 degrees
- moved C414 3.05 mm to (151.7, 108.7)
- moved C204 2.65 mm to (166.1, 54.4)
- moved C203 2.55 mm to (154.4, 66.3)
- moved C202 2.54 mm to (154.4, 71.1)
- moved C205 2.41 mm to (154.4, 54.4)
- moved C207 2.30 mm to (166.1, 62.2)
- moved C501 2.29 mm to (141.0, 68.3)
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Routing:
- net GND: track 112.2 -> 119.6 mm, vias 50 -> 47
- net /USB_to_UART/USB_LED_0: track 8.35 -> 15.5 mm
- net +3V3: track 78.0 -> 84.8 mm, vias 34 -> 32
- net /USB_to_UART/USB_LED_1: track 10.6 -> 17.0 mm
- net /Memory/EPI0S28: track 26.8 -> 25.2 mm
- net /TM4C129/ETH_LED0: track 50.4 -> 52.0 mm
- net /TM4C129/~RST: track 34.5 -> 35.7 mm
- net Net-(R503-Pad2): track 6.96 -> 5.75 mm
- net Net-(C502-Pad1): track 3.31 -> 4.27 mm
- net /TM4C129/R_BIAS: track 1.95 -> 2.73 mm, vias 0 -> 1
- net /USB_to_UART/DBG_USB_SHIELD: track 4.19 -> 4.95 mm
- net /TM4C129/USER_LED3: track 40.5 -> 39.7 mm
- net /TM4C129/USER_LED0: track 31.8 -> 31.0 mm
- net /TM4C129/USER_LED1: track 34.7 -> 33.9 mm
- net /TM4C129/USER_LED2: track 37.5 -> 36.8 mm

Commit message: layout cleanup, updating pdf.
Routing:
- net /TM4C129/ETH_LED1: track 51.3 -> 46.8 mm
- net /TM4C129/ETH_LED0: track 52.0 -> 47.9 mm
- net GND: track 119.6 -> 117.9 mm, vias 47 -> 46

Commit message: finished layout. generated gerbers.
Parts:
- moved D402 14.9 mm to (174.9, 82.9)
- moved R205 14.9 mm to (136.8, 91.0)
- moved C207 14.9 mm to (153.0, 69.4)
- moved D407 14.9 mm to (174.9, 70.2)
- moved C201 14.9 mm to (153.0, 73.5)
- moved C204 14.9 mm to (153.0, 61.5)
- moved C206 14.9 mm to (153.0, 78.3)
- moved C403 14.9 mm to (147.5, 101.0)
- moved C404 14.9 mm to (159.4, 88.7)
- moved C406 14.9 mm to (159.4, 90.5)
- moved C408 14.9 mm to (159.4, 92.2)
- moved C411 14.9 mm to (157.9, 98.6)
- moved C412 14.9 mm to (157.9, 101.9)
- moved C502 14.9 mm to (133.0, 68.6)
- moved D403 14.9 mm to (174.9, 77.8)
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Other:
- rule trace_min: 0.127 -> 0.1524
- rule via_min_size: 0.4572 -> 0.508

Commit message: added board/company name
Other:
- board text added: "Raptor2000-A BAD Robotics"
Changed lines of the file:
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@@
   (general
     (thickness 1.6)
-    (drawings 4)
+    (drawings 5)
     (tracks 1205)
     (zones 0)
@@
     )
   )
+  (gr_text "Raptor2000-A\nBAD Robotics" (at 173.99 84.455 270) (layer F.SilkS)
+    (effects (font (size 1.5 1.5) (thickness 0.3)) (justify left))
+  )
   (gr_line (start 177.419 57.9755) (end 113.919 57.9755) (layer Edge.Cuts) (width 0.15))
